Commit message: add:works in risk countours

File: assets/urdf/heart1/heart.urdf (robot description, URDF)
Before this commit: robot heart, 1 links, 0 joints
Links:
- link base_link: geometry collision mesh filename=heart1.stl scale=1 1 1; visual mesh filename=heart1.stl scale=1 1 1

File: assets/urdf/heart2/heart.urdf (robot description, URDF)
Before this commit: robot heart, 1 links, 0 joints
Links:
- link base_link: geometry collision mesh filename=heart2.stl scale=1 1 1; visual mesh filename=heart2.stl scale=1 1 1
